File: onekey/onekey.kicad_pcb (KiCad board)
At the start: 2 copper layers, 28.4 x 22.6 mm, 6 parts, among them J1 Conn_01x04_Socket, SW1 SW_Push, U1 MOUDLE-SEEEDUINO-XIAO

Commit message: djahfj
Parts:
- C1: moved to F.Cu
- J1: moved to B.Cu
- moved J1 23.1 mm to (137.5, 109.0)
- moved C1 11.1 mm to (152.5, 94.1), turned to 0 degrees
Routing:
- net +5V: track 66.0 -> 43.0 mm
- net GND: track 57.0 -> 44.7 mm
- net EC11B: track 23.3 -> 32.9 mm
- net BACKLIGHT_LED: track 21.9 -> 14.9 mm
- net ENCODER_B: track 21.3 -> 26.8 mm
- net ENCODER_A: track 22.0 -> 26.1 mm
